File: hw/Home Security PWA/Home Security PWA/Home Security PWA.kicad_pcb (KiCad board)
At the start: 2 copper layers, 42 parts, among them J1 1884340000, J10 1884340000, J11 1884340000, J12 1884340000, J13 1884340000, J14 1884340000, J15 1884340000, J16 1884340000, J17 1884340000, J18 1884340000, J19 1884340000, J2 1884340000, J20 1884340000, J21 1884340000, J22 1884340000, J23 1884340000, J24 1884340000, J25 1884340000, J26 1884340000, J27 1884340000, J28 1884340000, J29 1884340000, J3 1884340000, J4 1884340000, J5 Conn_01x10_Male, J6 Conn_01x10_Male, J7 1884340000, J8 1884340000, J9 1884340000, U1 ADS1115IDGS, U2 ADS1115IDGS, U3 MCP23017_SO

Commit message: Design and layout done.
Parts:
- added C1: .1uF, Capacitor_SMD:C_0805_2012Metric_Pad1.18x1.45mm_HandSolder, F.Cu at (140.6, 66.4)
- added C2: .1uF, Capacitor_SMD:C_0805_2012Metric_Pad1.18x1.45mm_HandSolder, F.Cu at (140.6, 72.4)
- added C3: .1uF, Capacitor_SMD:C_0805_2012Metric_Pad1.18x1.45mm_HandSolder, F.Cu at (151.3, 68.5)
- added J30: 1884340000, footprint:CONN4_1884340000_WED, F.Cu at (105.2, 147.8)
- J1, J2: value 1884340000 -> Conn_01x10_Pin; footprint foorprint:1884340000 -> footprint:PPTC101LFBN-RC
- J10, J11, J12, J13, J14, J15, J16, J17, J18, J19, J20, J21, J22, J23, J24, J25, J26, J27, J28, J29, J3, J4, J7, J8, J9: footprint foorprint:1884340000 -> footprint:CONN4_1884340000_WED
- J5, J6: value Conn_01x10_Male -> 1884340000; footprint foorprint:PPTC101LFBN-RC -> footprint:CONN4_1884340000_WED
- moved U3 102.2 mm to (158.8, 65.3)
- moved J27 97.8 mm to (125.5, 147.8)
- moved J3 92.6 mm to (95.0, 115.3)
- moved R4 92.3 mm to (149.9, 57.9), turned to -90 degrees
- moved R6 90.0 mm to (141.0, 57.9), turned to -90 degrees
- moved R5 89.9 mm to (143.9, 57.9), turned to -90 degrees
- moved R8 88.4 mm to (149.9, 52.6), turned to -90 degrees
- moved R3 88.1 mm to (146.8, 57.9), turned to -90 degrees
- moved J4 87.7 mm to (105.2, 115.3)
- moved J7 86.9 mm to (95.0, 131.6)
- moved R10 86.4 mm to (141.0, 52.6), turned to -90 degrees
- moved J6 86.2 mm to (125.5, 115.3)
- moved R9 86.2 mm to (143.9, 52.6), turned to -90 degrees
- moved J8 86.1 mm to (105.2, 131.6)
- moved J9 85.3 mm to (115.3, 131.6)
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Connections:
- J1 pad 1: /ADC1_0 -> +5V
- J1 pad 2: /ADC1_0 -> +3.3V
- J1 pad 4: GND -> unconnected-(J1-Pin_4-Pad4)
- J2 pad 1: /ADC1_1 -> unconnected-(J2-Pin_1-Pad1)
- J2 pad 2: /ADC1_1 -> unconnected-(J2-Pin_2-Pad2)
- J2 pad 3: GND -> unconnected-(J2-Pin_3-Pad3)
- J2 pad 4: GND -> unconnected-(J2-Pin_4-Pad4)
- J3 pad 1: /ADC1_2 -> /ADC0_0
- J3 pad 2: /ADC1_2 -> /ADC0_0
- J4 pad 1: /ADC1_3 -> /ADC0_1
- J4 pad 2: /ADC1_3 -> /ADC0_1
- J5 pad 1: +5V -> /ADC0_2
- J5 pad 2: +3.3V -> /ADC0_2
- J5 pad 4: unconnected-(J5-Pin_4-Pad4) -> GND
- J6 pad 1: unconnected-(J6-Pin_1-Pad1) -> /ADC0_3
- J6 pad 2: unconnected-(J6-Pin_2-Pad2) -> /ADC0_3
- J6 pad 3: unconnected-(J6-Pin_3-Pad3) -> GND
- J6 pad 4: unconnected-(J6-Pin_4-Pad4) -> GND
Routing:
- net +3.3V: track 0.00 -> 277.2 mm, vias 0 -> 13
- net /ADC1_0: track 0.00 -> 133.8 mm, vias 0 -> 1
- net /ADC1_1: track 0.00 -> 127.2 mm, vias 0 -> 1
- net /ADC1_2: track 0.00 -> 119.2 mm, vias 0 -> 1
- net /ADC0_0: track 0.00 -> 113.3 mm, vias 0 -> 1
- net /ADC1_3: track 0.00 -> 107.3 mm, vias 0 -> 1
- net /PB4: track 0.00 -> 103.8 mm, vias 0 -> 1
- net /ADC0_1: track 0.00 -> 103.8 mm, vias 0 -> 1
- net /PA0: track 0.00 -> 96.1 mm, vias 0 -> 1
- net /ADC0_2: track 0.00 -> 92.4 mm, vias 0 -> 1
- net /PB0: track 0.00 -> 92.3 mm, vias 0 -> 1
- net /PB5: track 0.00 -> 91.7 mm, vias 0 -> 1
- net /PA1: track 0.00 -> 83.0 mm, vias 0 -> 1
- net /SCL: track 0.00 -> 82.7 mm, vias 0 -> 3
- net /SDA: track 0.00 -> 82.2 mm, vias 0 -> 3
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- added copper zone on B.Cu, net GND
- added copper zone on F.Cu, net GND
Other:
- board outline added: 77.5 x 111.8 mm
- board text added: "+3.3V"
- board text added: "+5.0V"
- board text added: "1"
- board text added: "2"
- board text added: "A0_0"
- board text added: "A0_1"
- board text added: "A0_2"
- board text added: "A0_3"
- board text added: "A1_0"
- board text added: "A1_1"
- board text added: "A1_2"
- board text added: "A1_3"
- board text added: "ESP32-POE"
- board text added: "GND"
- board text added: "HOME SECURITY BREAKOUT BOARD"
- board text added: "PA0"
- board text added: "PA1"
- board text added: "PA2"
- board text added: "PA3"
- board text added: "PA4"
- board text added: "PA5"
- board text added: "PA6"
- board text added: "PA7"
- board text added: "PB0"
- board text added: "PB1"
- board text added: "PB2"
- board text added: "PB3"
- board text added: "PB4"
- board text added: "PB5"
- board text added: "PB6"
- board text added: "PB7"
