File: hw/Home Security PWA/Home Security PWA/Home Security PWA.kicad_sch (KiCad schematic)
At the start: 42 parts, among them J1 1884340000, J10 1884340000, J11 1884340000, J12 1884340000, J13 1884340000, J14 1884340000, J15 1884340000, J16 1884340000, J17 1884340000, J18 1884340000, J19 1884340000, J2 1884340000, J20 1884340000, J21 1884340000, J22 1884340000, J23 1884340000, J24 1884340000, J25 1884340000, J26 1884340000, J27 1884340000, J28 1884340000, J29 1884340000, J3 1884340000, J4 1884340000, J5 Conn_01x10_Male, J6 Conn_01x10_Male, J7 1884340000, J8 1884340000, J9 1884340000, U1 ADS1115IDGS, U2 ADS1115IDGS, U3 MCP23017_SO

Commit message: Design and layout done.
Parts:
- removed J2, J3: 1884340000, foorprint:1884340000, symbol 1884340000:1884340000
- removed J5, J6: Conn_01x10_Male, foorprint:PPTC101LFBN-RC, symbol Connector:Conn_01x10_Male
- added C1, C2, C3: .1uF, Capacitor_SMD:C_0805_2012Metric_Pad1.18x1.45mm_HandSolder, symbol Device:C_Small
- added J1, J2: Conn_01x10_Pin, footprint:PPTC101LFBN-RC, symbol Connector:Conn_01x10_Pin
- added J30, J5, J6: 1884340000, footprint:CONN4_1884340000_WED, symbol 1884340000:1884340000
- J10, J11, J12, J13, J14, J15, J16, J17, J18, J19, J20, J21, J22, J23, J24, J25, J26, J27, J28, J29, J4, J7, J8, J9: footprint foorprint:1884340000 -> footprint:CONN4_1884340000_WED
- J3: renamed from J1; footprint foorprint:1884340000 -> footprint:CONN4_1884340000_WED
Connections:
- net +3.3V: now also C1.1, C2.1, C3.1, J1.2 (Pin_2), J30.1, J30.2, J30.3, J30.4
- net +5V: now also J1.1 (Pin_1)
- net ADC0_0: now also J3.1, J3.2
- net ADC0_1: now also J4.1, J4.2
- net ADC0_2: now also J5.1, J5.2
- net ADC0_3: now also J6.1, J6.2
- net ADC1_0: no longer J3.1, J3.2
- net ADC1_3: no longer J4.1, J4.2
- net GND: now also C1.2, C2.2, C3.2, J1.3 (Pin_3), J5.3, J5.4, J6.3, J6.4
- net SCL: now also J2.6 (Pin_6)
- net SDA: now also J2.5 (Pin_5)
Other:
- note added: "HOME SECURITY BREAKOUT"
- moved on the sheet: J3, R1, R10, R2, R3, R4, R5, R6, R7, R8, R9, U1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
