File: hw/Home Security PWA/Home Security PWA.kicad_pcb (KiCad board)
At the start: 2 copper layers, 77.5 x 111.8 mm, 46 parts, among them J1 Conn_01x10_Pin, J10 1884340000, J11 1884340000, J12 1884340000, J13 1884340000, J14 1884340000, J15 1884340000, J16 1884340000, J17 1884340000, J18 1884340000, J19 1884340000, J2 Conn_01x10_Pin, J20 1884340000, J21 1884340000, J22 1884340000, J23 1884340000, J24 1884340000, J25 1884340000, J26 1884340000, J27 1884340000, J28 1884340000, J29 1884340000, J3 1884340000, J30 1884340000, J4 1884340000, J5 1884340000, J6 1884340000, J7 1884340000, J8 1884340000, J9 1884340000, U1 ADS1115IDGS, U2 ADS1115IDGS, U3 MCP23017_SO

Commit message: Rev A.
Added these "top" loader cable holders.
Added GPIOs that directly attach to the ESP32.
Parts:
- added J31: 1825960000, footprint:CONN_1825960000_WED, F.Cu at (95.2, 103.4)
- added J32: 1825960000, footprint:CONN_1825960000_WED, F.Cu at (105.4, 103.4)
- added J33: 1825960000, footprint:CONN_1825960000_WED, F.Cu at (115.6, 103.4)
- added J34: 1825960000, footprint:CONN_1825960000_WED, F.Cu at (125.7, 103.4)
- added SCL: TestPoint, TestPoint:TestPoint_THTPad_D2.0mm_Drill1.0mm, F.Cu at (166.2, 77.5)
- added SDA: TestPoint, TestPoint:TestPoint_THTPad_D2.0mm_Drill1.0mm, F.Cu at (162.1, 77.5)
- J10, J11, J12, J13, J14, J15, J16, J17, J18, J19, J20, J21, J22, J23, J24, J25, J26, J27, J28, J29, J3, J30, J4, J5, J6, J7, J8, J9: value 1884340000 -> 1825960000; footprint footprint:CONN4_1884340000_WED -> footprint:CONN_1825960000_WED
- moved R1 18.8 mm to (160.4, 102.1)
- moved R2 18.8 mm to (160.4, 105.1)
- moved J3 10.9 mm to (95.2, 126.2)
- moved J4 10.9 mm to (105.4, 126.2)
- moved J5 10.9 mm to (115.6, 126.2)
- moved J6 10.9 mm to (125.7, 126.2)
- moved J30 10.5 mm to (115.6, 149.1)
- moved J29 9.99 mm to (105.4, 149.1)
- moved J23 7.62 mm to (95.2, 91.9)
- moved J24 7.62 mm to (105.4, 91.9)
- moved J25 7.62 mm to (115.6, 91.9)
- moved J26 7.62 mm to (125.7, 91.9)
- moved J10 6.10 mm to (125.7, 137.7)
- moved J7 6.10 mm to (95.2, 137.7)
- moved J8 6.10 mm to (105.4, 137.7)
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Connections:
- J2 pad 10: unconnected-(J2-Pin_10-Pad10) -> /GPIO13
- J2 pad 7: unconnected-(J2-Pin_7-Pad7) -> /GPIO16
- J2 pad 8: unconnected-(J2-Pin_8-Pad8) -> /GPIO15
- J2 pad 9: unconnected-(J2-Pin_9-Pad9) -> /GPIO14
- J28 pad 3: +3.3V -> GND
- J28 pad 4: +3.3V -> GND
- J29 pad 1: +5V -> +3.3V
- J29 pad 2: +5V -> +3.3V
- J29 pad 3: +5V -> GND
- J29 pad 4: +5V -> GND
- J30 pad 1: +3.3V -> +5V
- J30 pad 2: +3.3V -> +5V
- J30 pad 3: +3.3V -> GND
- J30 pad 4: +3.3V -> GND
- U3 pad 18: unconnected-(U3-~{RESET}-Pad18) -> +3.3V
Routing:
- net /GPIO13: track 0.00 -> 91.5 mm, vias 0 -> 1
- net /GPIO14: track 0.00 -> 79.9 mm, vias 0 -> 1
- net /GPIO15: track 0.00 -> 68.2 mm, vias 0 -> 1
- net /GPIO16: track 0.00 -> 57.0 mm, vias 0 -> 1
- net +3.3V: track 277.2 -> 296.6 mm, vias 13 -> 17
- net /SCL: track 82.7 -> 97.5 mm, vias 3 -> 4
- net /ADC0_2: track 92.4 -> 107.0 mm
- net /ADC0_1: track 103.8 -> 117.6 mm
- net /ADC0_0: track 113.3 -> 127.1 mm
- net /ADC0_3: track 82.0 -> 95.7 mm
- net /SDA: track 82.2 -> 91.6 mm, vias 3 -> 4
- net /PA0: track 96.1 -> 86.8 mm
- net +5V: track 74.9 -> 65.7 mm
- net /PA1: track 83.0 -> 74.7 mm
- net /ADC1_0: track 133.8 -> 142.1 mm
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Other:
- board text added: "+"
- board text added: "-"
- board text added: "ANALOG INPUTS"
- board text added: "DIGITAL INPUTS"
- board text added: "IO13"
- board text added: "IO14"
- board text added: "IO15"
- board text added: "IO16"
- board text added: "REV A"
